File: hardware/lr2021-esp32s3/lr2021_esp32s3.kicad_pcb (KiCad board)
At the start: 4 copper layers, 90 x 65 mm, 84 parts, among them J1 USB-C, J2 5V IN, J3 3V3 IN, J4 GPIO, J5 SMA 915MHz, J6 SMA 2.4GHz, SW1 RESET, SW2 BOOT, U1 USBLC6-2SC6, U2 AP7361C-33E, U3 LM66100, U4 LM66100, U5 ESP32-S3-WROOM-1-N16R8, U6 LR2021IMLTRT, Y1 32MHz

Commit message: Route LR2021 + ESP32-S3 board; add fab outputs and build pipeline
- In2 becomes a +3V3 plane (L1 sig/RF, L2 GND, L3 3V3, L4 sig); every
  3V3/GND pad gets its own plane via
- Hand fanout of the LR2021 (crystal, NTC divider, SIMO loop, VBAT/VDCC/
  VPAX, SPI escape vias) and the duplicated USB-C pads; only DIO9 is used
  as IRQ (DIO7/8/11 freed to clear the QFN corner)
- Freerouting 1.9 routes the rest on L1/L4 (inner layers declared as power
  planes); single-layer vias removed, ~160 GND stitching vias added
- build.py: project -> schematic -> ERC -> PCB -> route (retried until DRC
  has no unconnected items) -> Gerbers/drill, JLCPCB BOM/CPL, PDFs, previews
- ERC: 0 errors (1 intentional LM66100 diode-OR warning)
  DRC with schematic parity: 0 errors, 0 unconnected, 0 parity issues

Co-Authored-By: Claude Opus 5.5 <noreply@anthropic.com>
Claude-Session: https://claude.ai/code/session_01GybN5CQfdUnddB4A81xgKu
Parts:
- moved SW2 37.5 mm to (143.0, 117.0)
- moved R7 23.4 mm to (139.5, 122.5)
- moved FB3 5.22 mm to (149.9, 131.2), turned to -90 degrees
- moved C5 5.00 mm to (119.0, 152.5)
- moved FB2 4.39 mm to (152.5, 128.8)
- moved C15 3.04 mm to (151.2, 131.2), turned to -90 degrees
- moved C13 2.62 mm to (153.8, 128.8)
- moved TH1 1.52 mm to (154.8, 123.4)
- moved U1 1.50 mm to (112.5, 125.5)
- moved L1 1.25 mm to (153.2, 132.4), turned to 180 degrees
- moved R8 1.00 mm to (154.8, 125.4)
- moved Y1 0.80 mm to (157.4, 124.0)
- moved C16 0.60 mm to (159.7, 122.6)
- moved FB1 0.42 mm to (153.5, 134.3)
- moved C12 0.36 mm to (155.0, 134.3), turned to -90 degrees
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Connections:
- U5 pad 12: /LR_DIO11 -> unconnected-(U5-IO8-Pad12)
- U5 pad 17: /LR_DIO7 -> unconnected-(U5-IO9-Pad17)
- U5 pad 25: /LR_DIO8 -> unconnected-(U5-IO48-Pad25)
- U6 pad 10: /LR_DIO8 -> unconnected-(U6-DIO8-Pad10)
- U6 pad 11: /LR_DIO7 -> unconnected-(U6-DIO7-Pad11)
- U6 pad 7: /LR_DIO11 -> unconnected-(U6-DIO11-Pad7)
Routing:
- net /GPIO4: track 0.00 -> 74.4 mm, vias 0 -> 1
- net /GPIO5: track 0.00 -> 66.0 mm, vias 0 -> 1
- net /GPIO16: track 0.00 -> 65.9 mm, vias 0 -> 1
- net /GPIO7: track 0.00 -> 65.8 mm, vias 0 -> 1
- net /GPIO15: track 0.00 -> 65.2 mm, vias 0 -> 1
- net /GPIO18: track 0.00 -> 63.8 mm, vias 0 -> 2
- net /GPIO6: track 0.00 -> 61.2 mm, vias 0 -> 2
- net /U0TXD: track 0.00 -> 61.2 mm, vias 0 -> 1
- net /GPIO17: track 0.00 -> 61.1 mm, vias 0 -> 2
- net /GPIO41: track 0.00 -> 59.0 mm, vias 0 -> 1
- net /U0RXD: track 0.00 -> 58.6 mm, vias 0 -> 1
- net /GPIO1: track 0.00 -> 55.4 mm, vias 0 -> 1
- net /GPIO42: track 0.00 -> 54.4 mm, vias 0 -> 1
- net /LR_NSS: track 0.00 -> 53.7 mm, vias 0 -> 2
- net /GPIO39: track 0.00 -> 51.0 mm, vias 0 -> 1
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- added copper zone on In2.Cu, net +3V3
- removed copper zone on In2.Cu, net GND
Other:
- board text added: "+"
- board text added: "-"
- board text added: "2.4 GHz"
- board text added: "3V3 IN"
- board text added: "5V IN"
- board text added: "915 MHz"
- board text added: "BOOT"
- board text added: "GPIO 1:3V3 2:5V 19,20:GND"
- board text added: "LR2021 + ESP32-S3 rev 1.0"
- board text added: "PWR"
- board text added: "RESET"
- board text added: "USB-C"
- board text added: "USR"
